File: AIL_LED_KICAD/AIL_LED.kicad_sch (KiCad schematic)
At the start: 22 parts, among them J1 Conn_01x02_Female

Commit message: updating with BOM
Parts:
- J1: footprint Connector 215760-1002:215760-YY02 -> Connector_Molex:Molex_Micro-Fit_3.0_43045-0200_2x01_P3.00mm_Horizontal
Changed lines of the file:
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@@
       (effects (font (size 1.27 1.27)) (justify left))
     )
-    (property "Footprint" "Connector 215760-1002:215760-YY02" (id 2) (at 133.985 46.355 0)
+    (property "Footprint" "Connector_Molex:Molex_Micro-Fit_3.0_43045-0200_2x01_P3.00mm_Horizontal" (id 2) (at 133.985 46.355 0)
       (effects (font (size 1.27 1.27)) hide)
     )
@@
     )
     (path "/6f1beb86-67e1-46bf-8c2b-6d1e1485d5c0"
-      (reference "J1") (unit 1) (value "Conn_01x02_Female") (footprint "Connector 215760-1002:215760-YY02")
+      (reference "J1") (unit 1) (value "Conn_01x02_Female") (footprint "Connector_Molex:Molex_Micro-Fit_3.0_43045-0200_2x01_P3.00mm_Horizontal")
     )
     (path "/facb0614-068b-4c9c-a466-d374df96a94c"
