File: AIL_MAIN_KICAD/AIL.kicad_sch (KiCad schematic)
At the start: 25 parts, among them IC1 LT8315, J1 Conn_01x02_Female, J2 Conn_01x02_Female

Commit message: Updating main board
Parts:
- removed J1: Conn_01x02_Female, 2155760-1002:215760-YY02, symbol Connector:Conn_01x02_Female
- added D10, D11, D12, D13, D14, D15, D16, D17, D18, D19, D20, D21, D22, D23, D24, D25, D26, D27, D28, D29, D5, D6, D7, D8, D9: LED, AIL_MAIN_FOOT:LEDC2012X100N, symbol Device:LED
- added R8: 20, Resistor_SMD:R_0603_1608Metric_Pad0.98x0.95mm_HandSolder, symbol Device:R
- J2: footprint 2155760-1002:215760-YY02 -> Connector_Molex:Molex_Micro-Fit_3.0_43045-0200_2x01_P3.00mm_Horizontal
Connections:
- net GND: now also D14.1 (K), D19.1 (K), D24.1 (K), D29.1 (K), D9.1 (K)
- net HV1: now also IC1.2 (DRAIN_2), IC1.3 (DRAIN_3)
- net ICGND: now also IC1.15 (GND_1)
- net 12V renamed +12V
- net +12V: now also R8.1
- new net: D8.1 (K), D9.2 (A)
- new net: D7.1 (K), D8.2 (A)
- new net: D6.1 (K), D7.2 (A)
- new net: D23.1 (K), D24.2 (A)
- new net: D12.1 (K), D13.2 (A)
- new net: D11.1 (K), D12.2 (A)
- new net: D5.1 (K), D6.2 (A)
- new net: D10.2 (A), D15.2 (A), D20.2 (A), D25.2 (A), D5.2 (A), R8.2
- new net: D28.1 (K), D29.2 (A)
- new net: D16.1 (K), D17.2 (A)
- new net: D15.1 (K), D16.2 (A)
- new net: D10.1 (K), D11.2 (A)
- new net: D27.1 (K), D28.2 (A)
- new net: D26.1 (K), D27.2 (A)
- new net: D22.1 (K), D23.2 (A)
- new net: D25.1 (K), D26.2 (A)
- new net: D13.1 (K), D14.2 (A)
- new net: D17.1 (K), D18.2 (A)
- new net: D18.1 (K), D19.2 (A)
- new net: D21.1 (K), D22.2 (A)
- new net: D20.1 (K), D21.2 (A)
- no-connect marks 4 -> 1
Other:
- moved on the sheet: C1, C2, C3, C4, C5, C6, C7, C8, C9, D1, D2, D4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

Commit message: updating with BOM
Parts:
- added C3: 22uF, Capacitor_SMD:C_0805_2012Metric_Pad1.18x1.45mm_HandSolder, symbol Device:C
- C1: footprint Capacitor_SMD:C_0603_1608Metric_Pad1.08x0.95mm_HandSolder -> Capacitor_SMD:C_1812_4532Metric_Pad1.57x3.40mm_HandSolder
- C2: value 43E-6 -> 22uF; footprint Capacitor_SMD:C_0603_1608Metric_Pad1.08x0.95mm_HandSolder -> Capacitor_SMD:C_0805_2012Metric_Pad1.18x1.45mm_HandSolder
- C4: footprint Capacitor_SMD:C_0603_1608Metric_Pad1.08x0.95mm_HandSolder -> Capacitor_SMD:C_01005_0402Metric_Pad0.57x0.30mm_HandSolder
- C9: value 100E-9 -> 10E-6
- R6: value 1.91E6 -> 1.87E6; footprint Resistor_SMD:R_0603_1608Metric_Pad0.98x0.95mm_HandSolder -> Capacitor_SMD:C_1206_3216Metric_Pad1.33x1.80mm_HandSolder
- renumbered C3 to C10
Connections:
- net +12V: now also C3.1
- net GND: now also C3.2
- net at IC1.17 (EN/UVLO), R6.1, R7.2: no longer C7.1
- net at D4.1 (K), R6.2: now also C7.1

Commit message: updating PCB with seperated BOMs
Parts:
- R2: footprint Resistor_SMD:R_0603_1608Metric_Pad0.98x0.95mm_HandSolder -> Resistor_SMD:R_1206_3216Metric_Pad1.30x1.75mm_HandSolder
- R5: footprint Resistor_SMD:R_0603_1608Metric_Pad0.98x0.95mm_HandSolder -> Resistor_SMD:R_2512_6332Metric_Pad1.40x3.35mm_HandSolder
Changed lines of the file:
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@@
     (property "Reference" "R5" (id 0) (at 214.63 50.8 90))
     (property "Value" "330E-3" (id 1) (at 214.63 53.34 90))
-    (property "Footprint" "Resistor_SMD:R_0603_1608Metric_Pad0.98x0.95mm_HandSolder" (id 2) (at 214.63 58.928 90)
+    (property "Footprint" "Resistor_SMD:R_2512_6332Metric_Pad1.40x3.35mm_HandSolder" (id 2) (at 214.63 58.928 90)
       (effects (font (size 1.27 1.27)) hide)
     )
@@
     (property "Reference" "R2" (id 0) (at 158.75 53.34 90))
     (property "Value" "10E3" (id 1) (at 158.75 55.88 90))
-    (property "Footprint" "Resistor_SMD:R_0603_1608Metric_Pad0.98x0.95mm_HandSolder" (id 2) (at 158.75 61.468 90)
+    (property "Footprint" "Resistor_SMD:R_1206_3216Metric_Pad1.30x1.75mm_HandSolder" (id 2) (at 158.75 61.468 90)
       (effects (font (size 1.27 1.27)) hide)
     )
@@
     )
     (path "/d847424d-7019-4df8-b961-1dd2d9facb89"
-      (reference "R2") (unit 1) (value "10E3") (footprint "Resistor_SMD:R_0603_1608Metric_Pad0.98x0.95mm_HandSolder")
+      (reference "R2") (unit 1) (value "10E3") (footprint "Resistor_SMD:R_1206_3216Metric_Pad1.30x1.75mm_HandSolder")
     )
     (path "/d5378109-6930-4bd2-ae9f-bf458fc3e1c0"
@@
     )
     (path "/6bdc0143-16b9-45a2-a52e-5ce15234cedb"
-      (reference "R5") (unit 1) (value "330E-3") (footprint "Resistor_SMD:R_0603_1608Metric_Pad0.98x0.95mm_HandSolder")
+      (reference "R5") (unit 1) (value "330E-3") (footprint "Resistor_SMD:R_2512_6332Metric_Pad1.40x3.35mm_HandSolder")
     )
     (path "/cddabd06-13bb-40e1-be82-10f94faf40c6"
